File: KabeltesterMEGA.kicad_pcb (KiCad board)
At the start: 2 copper layers, 93.5 x 80.5 mm, 65 parts, among them J1 Outputs, J2 Inputs, J3 LCD, J4 RotEnc, P1 Digital, P10 CONN_01X01, P11 CONN_01X01, P12 CONN_01X01, P13 CONN_01X01, P14 CONN_01X01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

Commit message: Fixed typo in B-SilkS
Parts:
- added QR1: oyvindskaaden/Cabletester, Logo:Github-SilkNonInv, B.Cu at (178.7, 100.7)
Other:
- board text added: "For schematics, code and documentation, scan QR or go to"
- board text added: "https://github.com/oyvindskaaden/Cabletester"
